File: schematics_and_pcbs/imac_g3_slot_loading_J22_adapter_board/imac_g3_slot_loading_J22_adapter_board.kicad_pcb (KiCad board)
At the start: 2 copper layers, 65 x 30 mm, 12 parts, among them J1 Conn_02x13_Odd_Even, J2 Screw_Terminal_01x10, J3 AudioJack3, J4 Conn_02x03_Odd_Even

Commit message: Use an in-stock capacitor in J22 board
Also add the regenerated gerbers
Parts:
- C1: footprint Capacitor_THT:CP_Radial_D4.0mm_P1.50mm -> Capacitor_THT:CP_Radial_D5.0mm_P2.00mm
- moved C1 1.00 mm to (167.8, 91.1)
Connections:
- J1 pad 12: Net-(J1-Pad12) -> unconnected-(J1-Pin_12-Pad12)
- J1 pad 21: Net-(J1-Pad21) -> unconnected-(J1-Pin_21-Pad21)
- J1 pad 22: Net-(J1-Pad22) -> unconnected-(J1-Pin_22-Pad22)
Routing:
- net Net-(JP2-B): track 37.6 -> 35.6 mm
- net Net-(JP1-B): track 15.0 -> 14.4 mm
Other:
- net class Default removed
